File: mcu.kicad_sch (KiCad schematic)
At the start: 12 parts, among them Q1 S8050, Q2 S8050, SW1 SW_Push, U4 ESP32-WROOM-32U

Commit message: start routing
Connections:
- net BUT1: now reaches U4.13 (IO14)
- net BUT0: now reaches U4.16 (IO13)
- net RDY: no longer names the net of U4.31 (IO19)
Changed lines of the file:
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@@
-    (effects (font (size 1.27 1.27)) (justify left))
-  )
-  (hierarchical_label "RDY" (shape input) (at 160.782 80.518 0) (fields_autoplaced)
     (effects (font (size 1.27 1.27)) (justify left))
   )
@@
     (effects (font (size 1.27 1.27)) (justify left))
   )
+  (hierarchical_label "BUT1" (shape input) (at 160.782 67.818 0) (fields_autoplaced)
+    (effects (font (size 1.27 1.27)) (justify left))
+  )
   (hierarchical_label "DATA" (shape input) (at 160.782 72.898 0) (fields_autoplaced)
     (effects (font (size 1.27 1.27)) (justify left))
@@
     (effects (font (size 1.27 1.27)) (justify left))
   )
+  (hierarchical_label "BUT0" (shape input) (at 160.782 65.278 0) (fields_autoplaced)
+    (effects (font (size 1.27 1.27)) (justify left))
+  )
