File: weighing_unit.kicad_sch (KiCad schematic)
At the start: 17 parts, among them Q3 MMBT3904, U5 LMV358, U6 ADS1115IDGS

Commit message: change dimensions
Parts:
- removed D3, D4, D6: BAT60A, Diode_SMD:D_SOD-323, symbol Diode:BAT60A
- removed Q3: MMBT3904, Package_TO_SOT_SMD:SOT-23, symbol Transistor_BJT:MMBT3904
- added D3, D4, D6: D_Zener, Diode_SMD:D_SMA, symbol Device:D_Zener
- added Q3: S8050, Package_TO_SOT_SMD:SOT-23, symbol Transistor_BJT:S8050
Connections:
- net 3V3: now also D3.1 (K)
- net GND: now also Q3.1 (E)
- net GNDA: now also D4.2 (A)
- net at BZ1.1 (+), R17.1: now also D6.1 (K)
- net at BZ1.2 (-): now also D6.2 (A), Q3.3 (C)
- net at R6.2, U6.4 (AIN0): now also D3.2 (A), D4.1 (K)
- net at R18.1: now also Q3.2 (B)
Changed lines of the file:
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@@
     )
   )
-  (symbol (lib_id "Diode:BAT60A") (at 106.426 101.346 270) (unit 1)
-    (in_bom yes) (on_board yes) (dnp no) (fields_autoplaced)
-    (property "Reference" "D6" (at 109.474 99.7585 90)
-      (effects (font (size 1.27 1.27)) (justify left))
-    )
-    (property "Value" "BAT60A" (at 109.474 102.2985 90)
-      (effects (font (size 1.27 1.27)) (justify left))
-    )
-    (property "Footprint" "Diode_SMD:D_SOD-323" (at 101.981 101.346 0)
-      (effects (font (size 1.27 1.27)) hide)
-    )
-    (property "Datasheet" "https://www.infineon.com/dgdl/Infineon-BAT60ASERIES-DS-v01_01-en.pdf?fileId=db3a304313d846880113def70c9304a9" (at 106.426 101.346 0)
-      (effects (font (size 1.27 1.27)) hide)
-    )
-    (pin "2")
-    (pin "1")
-    (instances
-      (project "scale"
-        (path "/8f227bf3-f4cf-485c-a746-8377af835d89/39c2c3b0-4826-42ca-a0df-7d76b180d9b9"
-          (reference "D6") (unit 1)
+  (symbol (lib_id "Device:D_Zener") (at 106.172 62.23 270) (unit 1)
+    (in_bom yes) (on_board yes) (dnp no) (fields_autoplaced)
+    (property "Reference" "D4" (at 108.966 60.96 90)
+      (effects (font (size 1.27 1.27)) (justify left))
+    )
+    (property "Value" "D_Zener" (at 108.966 63.5 90)
+      (effects (font (size 1.27 1.27)) (justify left))
+    )
+    (property "Footprint" "Diode_SMD:D_SMA" (at 106.172 62.23 0)
+      (effects (font (size 1.27 1.27)) hide)
+    )
+    (property "Datasheet" "~" (at 106.172 62.23 0)
+      (effects (font (size 1.27 1.27)) hide)
+    )
+    (pin "2")
+    (pin "1")
+    (instances
+      (project "scale"
+        (path "/8f227bf3-f4cf-485c-a746-8377af835d89/39c2c3b0-4826-42ca-a0df-7d76b180d9b9"
+          (reference "D4") (unit 1)
         )
       )
@@
     )
   )
-  (symbol (lib_id "Diode:BAT60A") (at 106.172 49.022 270) (unit 1)
-    (in_bom yes) (on_board yes) (dnp no) (fields_autoplaced)
-    (property "Reference" "D3" (at 109.22 47.4345 90)
-      (effects (font (size 1.27 1.27)) (justify left))
-    )
-    (property "Value" "BAT60A" (at 109.22 49.9745 90)
-      (effects (font (size 1.27 1.27)) (justify left))
-    )
-    (property "Footprint" "Diode_SMD:D_SOD-323" (at 101.727 49.022 0)
-      (effects (font (size 1.27 1.27)) hide)
-    )
-    (property "Datasheet" "https://www.infineon.com/dgdl/Infineon-BAT60ASERIES-DS-v01_01-en.pdf?fileId=db3a304313d846880113def70c9304a9" (at 106.172 49.022 0)
-      (effects (font (size 1.27 1.27)) hide)
-    )
-    (pin "2")
-    (pin "1")
-    (instances
-      (project "scale"
-        (path "/8f227bf3-f4cf-485c-a746-8377af835d89/39c2c3b0-4826-42ca-a0df-7d76b180d9b9"
-          (reference "D3") (unit 1)
-        )
-      )
-    )
-  )
   (symbol (lib_id "Device:R") (at 78.74 42.418 90) (unit 1)
     (in_bom yes) (on_board yes) (dnp no) (fields_autoplaced)
@@
     )
   )
+  (symbol (lib_id "Device:D_Zener") (at 106.172 49.022 270) (unit 1)
+    (in_bom yes) (on_board yes) (dnp no) (fields_autoplaced)
+    (property "Reference" "D3" (at 108.966 47.752 90)
+      (effects (font (size 1.27 1.27)) (justify left))
+    )
+    (property "Value" "D_Zener" (at 108.966 50.292 90)
+      (effects (font (size 1.27 1.27)) (justify left))
+    )
+    (property "Footprint" "Diode_SMD:D_SMA" (at 106.172 49.022 0)
+      (effects (font (size 1.27 1.27)) hide)
+    )
+    (property "Datasheet" "~" (at 106.172 49.022 0)
+      (effects (font (size 1.27 1.27)) hide)
+    )
+    (pin "2")
+    (pin "1")
+    (instances
+      (project "scale"
+        (path "/8f227bf3-f4cf-485c-a746-8377af835d89/39c2c3b0-4826-42ca-a0df-7d76b180d9b9"
+          (reference "D3") (unit 1)
+        )
+      )
+    )
+  )
   (symbol (lib_id "Device:R") (at 98.298 113.538 270) (unit 1)
     (in_bom yes) (on_board yes) (dnp no) (fields_autoplaced)
@@
     )
   )
-  (symbol (lib_id "Transistor_BJT:MMBT3904") (at 109.474 113.538 0) (unit 1)
-    (in_bom yes) (on_board yes) (dnp no) (fields_autoplaced)
-    (property "Reference" "Q3" (at 115.57 112.268 0)
-      (effects (font (size 1.27 1.27)) (justify left))
-    )
-    (property "Value" "MMBT3904" (at 115.57 114.808 0)
-      (effects (font (size 1.27 1.27)) (justify left))
-    )
-    (property "Footprint" "Package_TO_SOT_SMD:SOT-23" (at 114.554 115.443 0)
-      (effects (font (size 1.27 1.27) italic) (justify left) hide)
-    )
-    (property "Datasheet" "https://www.onsemi.com/pdf/datasheet/pzt3904-d.pdf" (at 109.474 113.538 0)
-      (effects (font (size 1.27 1.27)) (justify left) hide)
-    )
-    (pin "3")
-    (pin "1")
-    (pin "2")
-    (instances
-      (project "scale"
-        (path "/8f227bf3-f4cf-485c-a746-8377af835d89/39c2c3b0-4826-42ca-a0df-7d76b180d9b9"
-          (reference "Q3") (unit 1)
-        )
-      )
-    )
-  )
   (symbol (lib_id "power:GND") (at 147.32 43.942 0) (unit 1)
     (in_bom yes) (on_board yes) (dnp no) (fields_autoplaced)
@@
         (path "/8f227bf3-f4cf-485c-a746-8377af835d89/39c2c3b0-4826-42ca-a0df-7d76b180d9b9"
           (reference "C5") (unit 1)
-        )
-      )
-    )
-  )
-  (symbol (lib_id "Diode:BAT60A") (at 106.172 62.23 270) (unit 1)
-    (in_bom yes) (on_board yes) (dnp no) (fields_autoplaced)
-    (property "Reference" "D4" (at 109.22 60.6425 90)
-      (effects (font (size 1.27 1.27)) (justify left))
-    )
-    (property "Value" "BAT60A" (at 109.22 63.1825 90)
-      (effects (font (size 1.27 1.27)) (justify left))
-    )
-    (property "Footprint" "Diode_SMD:D_SOD-323" (at 101.727 62.23 0)
-      (effects (font (size 1.27 1.27)) hide)
-    )
-    (property "Datasheet" "https://www.infineon.com/dgdl/Infineon-BAT60ASERIES-DS-v01_01-en.pdf?fileId=db3a304313d846880113def70c9304a9" (at 106.172 62.23 0)
-      (effects (font (size 1.27 1.27)) hide)
-    )
-    (pin "2")
-    (pin "1")
-    (instances
-      (project "scale"
-        (path "/8f227bf3-f4cf-485c-a746-8377af835d89/39c2c3b0-4826-42ca-a0df-7d76b180d9b9"
-          (reference "D4") (unit 1)
         )
       )
@@
     )
   )
+  (symbol (lib_id "Device:D_Zener") (at 106.426 101.346 270) (unit 1)
+    (in_bom yes) (on_board yes) (dnp no) (fields_autoplaced)
+    (property "Reference" "D6" (at 109.22 100.076 90)
+      (effects (font (size 1.27 1.27)) (justify left))
+    )
+    (property "Value" "D_Zener" (at 109.22 102.616 90)
+      (effects (font (size 1.27 1.27)) (justify left))
+    )
+    (property "Footprint" "Diode_SMD:D_SMA" (at 106.426 101.346 0)
+      (effects (font (size 1.27 1.27)) hide)
+    )
+    (property "Datasheet" "~" (at 106.426 101.346 0)
+      (effects (font (size 1.27 1.27)) hide)
+    )
+    (pin "2")
+    (pin "1")
+    (instances
+      (project "scale"
+        (path "/8f227bf3-f4cf-485c-a746-8377af835d89/39c2c3b0-4826-42ca-a0df-7d76b180d9b9"
+          (reference "D6") (unit 1)
+        )
+      )
+    )
+  )
   (symbol (lib_id "Amplifier_Operational:LMV358") (at 80.01 55.626 0) (unit 1)
     (in_bom yes) (on_board yes) (dnp no) (fields_autoplaced)
@@
         )
       )
+    )
+  )
+  (symbol (lib_id "Transistor_BJT:S8050") (at 109.474 113.538 0) (unit 1)
+    (in_bom yes) (on_board yes) (dnp no) (fields_autoplaced)
+    (property "Reference" "Q3" (at 114.554 112.268 0)
+      (effects (font (size 1.27 1.27)) (justify left))
+    )
+    (property "Value" "S8050" (at 114.554 114.808 0)
+      (effects (font (size 1.27 1.27)) (justify left))
+    )
+    (property "Footprint" "Package_TO_SOT_SMD:SOT-23" (at 114.554 115.443 0)
+      (effects (font (size 1.27 1.27) italic) (justify left) hide)
+    )
+    (property "Datasheet" "http://www.unisonic.com.tw/datasheet/S8050.pdf" (at 109.474 113.538 0)
+      (effects (font (size 1.27 1.27)) (justify left) hide)
+    )
+    (pin "1")
+    (pin "2")
+    (pin "3")
+    (instances
+      (project "scale"
+        (path "/8f227bf3-f4cf-485c-a746-8377af835d89/39c2c3b0-4826-42ca-a0df-7d76b180d9b9"
+          (reference "Q3") (unit 1)
+        )
+      )
