File: power_management.kicad_sch (KiCad schematic)
At the start: 0 parts

Commit message: add mcu, sensor, sensor inst, power
Parts:
- added C1, C2: 100u, Capacitor_SMD:CP_Elec_6.3x5.7, symbol Device:C_Polarized
- added C3: 1u, Capacitor_SMD:C_0805_2012Metric, symbol Device:C
- added C4: 100n, Capacitor_SMD:C_0805_2012Metric, symbol Device:C
- added D1: D_Zener, Diode_SMD:D_SMA, symbol Device:D_Zener
- added D2: LED, LED_SMD:LED_0805_2012Metric, symbol Device:LED
- added F1: Fuse, LED_SMD:LED_0805_2012Metric, symbol Device:Fuse
- added L1: 100u, BBG:IND_CDRH127-LDNP-470MC_SUM, symbol Device:L
- added R1: 3k3, Resistor_SMD:R_0805_2012Metric, symbol Device:R
- added U1: HLK-10M12, BBG:HLK-10_HLK, symbol BBG:HLK-10M12
- added U2: LM2576HVS-5, Package_TO_SOT_SMD:TO-263-5_TabPin3, symbol Regulator_Switching:LM2576HVS-5
- added U3: AMS1117-3.3, Package_TO_SOT_SMD:SOT-223-3_TabPin2, symbol Regulator_Linear:AMS1117-3.3
Connections:
- new net: D1.1 (K), L1.1, U2.2 (OUT)
- new net: C1.1, F1.2, U2.1 (VIN)
- new net: D2.1 (K), R1.1
- new net: F1.1, U1.4 (+VO)
- new net 3V3: C4.1, D2.2 (A), U3.2 (VO)
- new net 5V: C2.1, C3.1, L1.2, U2.4 (FB), U3.3 (VI)
- new net AC_1: U1.1 (AC)
- new net AC_2: U1.2 (AC)
- new net GND: C1.2, C2.2, C3.2, C4.2, D1.2 (A), R1.2, U1.3 (-V0), U2.3 (GND), U2.5 (~{ON}/OFF), U3.1 (GND)

Commit message: add footprint and step
Parts:
- F1: footprint LED_SMD:LED_0805_2012Metric -> Fuse:Fuse_1206_3216Metric
Changed lines of the file:
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@@
       (effects (font (size 1.27 1.27)))
     )
-    (property "Footprint" "LED_SMD:LED_0805_2012Metric" (at 127 64.262 90)
+    (property "Footprint" "Fuse:Fuse_1206_3216Metric" (at 127 64.262 90)
       (effects (font (size 1.27 1.27)) hide)
     )
